Commit message: Add xml linter

File: test/rrr.urdf.xacro (robot description, xacro)
@@ -1,16 +1,16 @@
-<?xml version="1.0"?>
+<?xml version="1.0" ?>
 <robot xmlns:xacro="http://www.ros.org/wiki/xacro" name="rrr_robot">
   <link name="base_link">
     <visual>
       <geometry>
-        <cylinder length="0.05" radius="0.1"/>
+        <cylinder length="0.05" radius="0.1" />
       </geometry>
       <material name="blue">
-        <color rgba="0 0 0.8 1"/>
+        <color rgba="0 0 0.8 1" />
       </material>
     </visual>
     <collision>
       <geometry>
-        <cylinder length="0.05" radius="0.1"/>
+        <cylinder length="0.05" radius="0.1" />
       </geometry>
     </collision>
@@ -19,16 +19,16 @@
     <visual>
       <geometry>
-        <box size="0.1 0.1 0.5"/>
+        <box size="0.1 0.1 0.5" />
       </geometry>
-      <origin xyz="0 0 0.25" rpy="0 0 0"/>
+      <origin xyz="0 0 0.25" rpy="0 0 0" />
       <material name="red">
-        <color rgba="0.8 0 0 1"/>
+        <color rgba="0.8 0 0 1" />
       </material>
     </visual>
     <collision>
       <geometry>
-        <box size="0.1 0.1 0.5"/>
+        <box size="0.1 0.1 0.5" />
       </geometry>
-      <origin xyz="0 0 0.25" rpy="0 0 0"/>
+      <origin xyz="0 0 0.25" rpy="0 0 0" />
     </collision>
   </link>
@@ -36,16 +36,16 @@
     <visual>
       <geometry>
-        <box size="0.1 0.1 0.4"/>
+        <box size="0.1 0.1 0.4" />
       </geometry>
-      <origin xyz="0 0 0.2" rpy="0 0 0"/>
+      <origin xyz="0 0 0.2" rpy="0 0 0" />
       <material name="green">
-        <color rgba="0 0.8 0 1"/>
+        <color rgba="0 0.8 0 1" />
       </material>
     </visual>
     <collision>
       <geometry>
-        <box size="0.1 0.1 0.4"/>
+        <box size="0.1 0.1 0.4" />
       </geometry>
-      <origin xyz="0 0 0.2" rpy="0 0 0"/>
+      <origin xyz="0 0 0.2" rpy="0 0 0" />
     </collision>
   </link>
@@ -53,16 +53,16 @@
     <visual>
       <geometry>
-        <box size="0.1 0.1 0.3"/>
+        <box size="0.1 0.1 0.3" />
       </geometry>
-      <origin xyz="0 0 0.15" rpy="0 0 0"/>
+      <origin xyz="0 0 0.15" rpy="0 0 0" />
       <material name="yellow">
-        <color rgba="0.8 0.8 0 1"/>
+        <color rgba="0.8 0.8 0 1" />
       </material>
     </visual>
     <collision>
       <geometry>
-        <box size="0.1 0.1 0.3"/>
+        <box size="0.1 0.1 0.3" />
       </geometry>
-      <origin xyz="0 0 0.15" rpy="0 0 0"/>
+      <origin xyz="0 0 0.15" rpy="0 0 0" />
     </collision>
   </link>
@@ -70,43 +70,43 @@
     <visual>
       <geometry>
-        <sphere radius="0.05"/>
+        <sphere radius="0.05" />
       </geometry>
       <material name="white">
-        <color rgba="1 1 1 1"/>
+        <color rgba="1 1 1 1" />
       </material>
     </visual>
     <collision>
       <geometry>
-        <sphere radius="0.05"/>
+        <sphere radius="0.05" />
       </geometry>
     </collision>
   </link>
   <joint name="joint1" type="revolute">
-    <parent link="base_link"/>
-    <child link="link1"/>
-    <origin xyz="0 0 0.025" rpy="0 0 0"/>
-    <axis xyz="0 0 1"/>
-    <limit lower="-3.14159" upper="3.14159" effort="100" velocity="1"/>
+    <parent link="base_link" />
+    <child link="link1" />
+    <origin xyz="0 0 0.025" rpy="0 0 0" />
+    <axis xyz="0 0 1" />
+    <limit lower="-3.14159" upper="3.14159" effort="100" velocity="1" />
   </joint>
   <joint name="joint2" type="revolute">
-    <parent link="link1"/>
-    <child link="link2"/>
-    <origin xyz="0 0 0.5" rpy="0 0 0"/>
-    <axis xyz="0 1 0"/>
-    <limit lower="-3.14159" upper="3.14159" effort="100" velocity="1"/>
+    <parent link="link1" />
+    <child link="link2" />
+    <origin xyz="0 0 0.5" rpy="0 0 0" />
+    <axis xyz="0 1 0" />
+    <limit lower="-3.14159" upper="3.14159" effort="100" velocity="1" />
   </joint>
   <joint name="joint3" type="revolute">
-    <parent link="link2"/>
-    <child link="link3"/>
-    <origin xyz="0 0 0.4" rpy="0 0 0"/>
-    <axis xyz="0 1 0"/>
-    <limit lower="-3.14159" upper="3.14159" effort="100" velocity="1"/>
+    <parent link="link2" />
+    <child link="link3" />
+    <origin xyz="0 0 0.4" rpy="0 0 0" />
+    <axis xyz="0 1 0" />
+    <limit lower="-3.14159" upper="3.14159" effort="100" velocity="1" />
   </joint>
   <joint name="end_effector_joint" type="revolute">
-    <parent link="link3"/>
-    <child link="end_effector"/>
-    <origin xyz="0 0 0.3" rpy="0 0 0"/>
-    <axis xyz="0 0 1"/>
-    <limit lower="0" upper="0" effort="0" velocity="0"/>
+    <parent link="link3" />
+    <child link="end_effector" />
+    <origin xyz="0 0 0.3" rpy="0 0 0" />
+    <axis xyz="0 0 1" />
+    <limit lower="0" upper="0" effort="0" velocity="0" />
   </joint>
   <ros2_control name="name" type="system">
@@ -117,23 +117,23 @@
     </hardware>
     <joint name="joint_1">
-      <command_interface name="position"/>
+      <command_interface name="position" />
       <state_interface name="position">
         <param name="initial_value">0.2</param>
       </state_interface>
-      <state_interface name="velocity"/>
+      <state_interface name="velocity" />
     </joint>
     <joint name="joint_2">
-      <command_interface name="position"/>
+      <command_interface name="position" />
       <state_interface name="position">
         <param name="initial_value">0.3</param>
       </state_interface>
-      <state_interface name="velocity"/>
+      <state_interface name="velocity" />
     </joint>
     <joint name="joint_3">
-      <command_interface name="position"/>
+      <command_interface name="position" />
       <state_interface name="position">
         <param name="initial_value">0.1</param>
       </state_interface>
-      <state_interface name="velocity"/>
+      <state_interface name="velocity" />
     </joint>
   </ros2_control>

Commit message: Fix joint names

File: test/rrr.urdf.xacro (robot description, xacro)
@@ -82,5 +82,5 @@
     </collision>
   </link>
-  <joint name="joint1" type="revolute">
+  <joint name="joint_1" type="revolute">
     <parent link="base_link" />
     <child link="link1" />
@@ -89,5 +89,5 @@
     <limit lower="-3.14159" upper="3.14159" effort="100" velocity="1" />
   </joint>
-  <joint name="joint2" type="revolute">
+  <joint name="joint_2" type="revolute">
     <parent link="link1" />
     <child link="link2" />
@@ -96,5 +96,5 @@
     <limit lower="-3.14159" upper="3.14159" effort="100" velocity="1" />
   </joint>
-  <joint name="joint3" type="revolute">
+  <joint name="joint_3" type="revolute">
     <parent link="link2" />
     <child link="link3" />
